Commit message: Strengthen Hall of Mirrors causal evidence

File: containers/harbor/mirrors_robot.urdf (robot description, URDF)
Before this commit: robot entryplug_hall_of_mirrors, 8 links, 7 joints
Links:
- added link spectator_camera_mujoco_frame
Joints:
- added joint spectator_camera_joint: type fixed, parent world, child spectator_camera_mujoco_frame, origin xyz=3.6 1.25 3.0
